File: Headphones.kicad_pcb (KiCad board)
At the start: 2 copper layers, 1 part, among them U1 MOUDLE-SEEEDUINO-XIAO-ESP32C3

Commit message: Amp
Parts:
- U1: footprint Arduino:MOUDLE14P-SMD-2.54-21X17.8MM -> arduino-library:MOUDLE14P-SMD-2.54-21X17.8MM
- moved U1 6.92 mm to (136.6, 99.1)
