File: Headphones.kicad_sch (KiCad schematic)
At the start: 1 part, among them U1 MOUDLE-SEEEDUINO-XIAO-ESP32C3

Commit message: Amp
Parts:
- added IC1: MAX98306ETD+T, SON40P300X300X80-15N, symbol SamacSys_Parts:MAX98306ETD+T
- added J1: Conn_01x02_Pin, symbol Connector:Conn_01x02_Pin
- U1: footprint Arduino:MOUDLE14P-SMD-2.54-21X17.8MM -> arduino-library:MOUDLE14P-SMD-2.54-21X17.8MM
Connections:
- net at U1.15 (BAT+): now also J1.1 (Pin_1)
- net at U1.16 (BAT-): now also J1.2 (Pin_2)
Other:
- moved on the sheet: U1
